File: hw/barbecue/barbecue.kicad_sch (KiCad schematic)
At the start: 52 parts, among them J1 47590-0001, J10 TFT, J11 SDCard, J2 Screw_Terminal_01x02, J3 bootsel, J4 gnd clk swd, J5 +pwm3-, J6 R_{ntc}, J7 +pwm2-, J8 +pwm1-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

Commit message: Fix board PWM outputs
Signed-off-by: Jan Hamal Dvořák <mordae@anilinux.org>
Parts:
- removed Q1, Q3, Q5: AO3401A, Package_TO_SOT_SMD:SOT-23, symbol Device:Q_PMOS_GSD
- removed Q6: AO3400A, Package_TO_SOT_SMD:SOT-23, symbol Device:Q_NMOS_GSD
- removed R1, R11, R12: 47k, Resistor_SMD:R_0402_1005Metric, symbol Device:R_Small
- added Q3: AO3400A, Package_TO_SOT_SMD:SOT-23, symbol Device:Q_NMOS_GSD
- J7: value +pwm2- -> +pwm3-
- J8: value +pwm1- -> +pwm3-
Connections:
- net +5V: now also J5.1 (Pin_1), J7.1 (Pin_1), J8.1 (Pin_1); no longer R8.1
- net GND: now also R8.2, Q3.2 (S); no longer J5.2 (Pin_2), J7.2 (Pin_2), J8.2 (Pin_2)
- net at Q2.3 (D): now also J5.2 (Pin_2); no longer J5.1 (Pin_1)
- net at Q4.3 (D): now also J8.2 (Pin_2); no longer J7.1 (Pin_1)
- net pwm1a renamed PWM_{1}
- net PWM_{1}: now also Q4.1 (G), R9.1
- net pwm1b: no longer names the net of U2.3 (GPIO1)
- removed net pwm2a: Q4.1 (G), R9.1, U2.4 (GPIO2)
- net pwm2b: no longer names the net of U2.5 (GPIO3)
- net pwm2b: no longer R8.2
- net pwm3a renamed PWM_{3}
- net pwm3b: no longer names the net of U2.7 (GPIO5)
- new net: J7.2 (Pin_2), Q3.3 (D)
- new net PWM_{2}: Q3.1 (G), R8.1, U2.4 (GPIO2)
- no-connect marks 22 -> 25
Other:
- moved on the sheet: J5, Q2, R2

Commit message: Version 1.1 as sent to manufacturing
Signed-off-by: Jan Hamal Dvořák <mordae@anilinux.org>
Parts:
- removed J10: TFT, Connector_PinSocket_2.54mm:PinSocket_1x11_P2.54mm_Vertical, symbol Connector_Generic:Conn_01x11
- removed J11: SDCard, Connector_PinSocket_2.54mm:PinSocket_1x04_P2.54mm_Vertical, symbol Connector_Generic:Conn_01x04
- removed J9: OLED, Connector_PinSocket_2.54mm:PinSocket_1x04_P2.54mm_Vertical, symbol Connector_Generic:Conn_01x04
- added C11, C12: 22u, Capacitor_SMD:C_0603_1608Metric, symbol Device:C_Small
- added H8: Tooling, Barbecue:ToolingHole, symbol Mechanical:MountingHole
- added U4: ILI9225-MOD, Barbecue:ILI9225-MOD, symbol Barbecue:ILI9225-MOD
- J5: value +pwm3- -> +HEAT-
- J6: value R_{ntc} -> NTC
- J7: value +pwm3- -> +FAN1-
- J8: value +pwm3- -> +FAN2-
- R10: footprint Resistor_SMD:R_0402_1005Metric -> Resistor_SMD:R_0603_1608Metric
Connections:
- net tft_sclk is gone; now on net re_b: U2.13 (GPIO10)
- net +3V3: now also C12.1, U4.1 (VCC)
- net +5V: now also C11.1
- net GND: now also C11.2, C12.2, U4.2 (GND), U4.3 (GND)
- net re_a: now also U2.12 (GPIO9); no longer U2.37 (GPIO25)
- net re_b: no longer U2.36 (GPIO24)
- net re_sw: now also U2.14 (GPIO11); no longer U2.35 (GPIO23)
- net tft_cs: now also U2.32 (GPIO21), U4.11 (CS); no longer U2.12 (GPIO9)
- net tft_mosi: now also U2.35 (GPIO23), U4.8 (SDA); no longer U2.14 (GPIO11)
- net tft_rs: now also U2.36 (GPIO24), U4.9 (RS); no longer U2.17 (GPIO14)
- net tft_rst: now also U2.37 (GPIO25), U4.10 (RST); no longer U2.11 (GPIO8)
- net tsense: now also U2.40 (GPIO28_ADC2); no longer U2.41 (GPIO29_ADC3)
- net sd_cs: now reaches U2.3 (GPIO1)
- net sd_cs: now also U4.12 (CS)
- net tft_sck: now reaches U2.34 (GPIO22)
- net tft_sck: now also U4.7 (CLK)
- net fan2: now reaches U2.38 (GPIO26_ADC0)
- net fan2: now also Q4.1 (G), R9.1
- net fan1: now reaches U2.39 (GPIO27_ADC1)
- net fan1: now also Q3.1 (G), R8.1
- net sd_mosi: now reaches U2.5 (GPIO3)
- net sd_mosi: now also U4.13 (MOSI)
- removed net PWM_{1}: Q4.1 (G), R9.1, U2.2 (GPIO0)
- removed net PWM_{2}: Q3.1 (G), R8.1, U2.4 (GPIO2)
- net PWM_{3} renamed heat
- net heat: now also U2.41 (GPIO29_ADC3); no longer U2.6 (GPIO4)
- net scl: no longer names the net of U2.9 (GPIO7)
- net sda: no longer names the net of U2.8 (GPIO6)
- new net sd_miso: U2.6 (GPIO4), U4.15 (MISO)
- new net sd_sck: U2.4 (GPIO2), U4.14 (SCK)
- no-connect marks 25 -> 16
Other:
- moved on the sheet: SW1
